Commit message: better xacro

File: fake_car.urdf.xacro (robot description, xacro)
@@ -3,33 +3,39 @@
   <xacro:property name="wheel_radius" value="0.056"/>
   <xacro:property name="wheel_width" value="0.047"/>
+  <xacro:property name="wheel_friction" value="0.8"/>
   <xacro:property name="wheelbase_length" value="0.3429"/>
   <xacro:property name="front_wheelbase_width" value="0.25"/>
   <xacro:property name="rear_wheelbase_width" value="0.25"/>
   <xacro:property name="wheel_mass" value="0.1"/>
-  <macro name="cylinder_inertia" params="m r h">
+  <xacro:property name="total_mass" value = "3.0"/>
+  <xacro:property name="chassis_height" value = "0.06"/>
+  <xacro:property name="chassis_elevation" value = "0.03"/>
+  <xacro:property name="chassis_mass" value = "${total_mass-4*wheel_mass}"/>
+  <xacro:macro name="cylinder_inertia" params="m r h">
         <inertia  ixx="${m*(3*r*r+h*h)/12}" ixy = "0" ixz = "0"
                     iyy="${m*(3*r*r+h*h)/12}" iyz = "0"
                     izz="${m*r*r/2}" />
-  </macro>
-  <macro name="box_inertia" params="m x y z">
+  </xacro:macro>
+  <xacro:macro name="box_inertia" params="m x y z">
           <inertia  ixx="${m*(y*y+z*z)/12}" ixy = "0" ixz = "0"
                     iyy="${m*(x*x+z*z)/12}" iyz = "0"
                     izz="${m*(x*x+z*z)/12}" />
-  </macro>
-  <macro name="sphere_inertia" params="m r">
+  </xacro:macro>
+  <xacro:macro name="sphere_inertia" params="m r">
           <inertia  ixx="${2*m*r*r/5}" ixy = "0" ixz = "0"
                     iyy="${2*m*r*r/5}" iyz = "0"
                     izz="${2*m*r*r/5}" />
-  </macro>
-  <macro name="cylinder_inertial" params="m r h">
+  </xacro:macro>
+  <xacro:macro name="cylinder_inertial" params="m r h">
     <inertial>
       <mass value="${m}"/>
-      <xacro:cylinder_inertia m="${m}" r="${r}" h="${h}"/>
-    </inertial>
-  </macro>
+      <cylinder_inertia m="${m}" r="${r}" h="${h}"/>
+    </inertial>
+  </xacro:macro>
   <link name="base_link">
     <visual>
-      <geometry>
-        <cylinder length="0.02" radius="0.01"/>
+      <origin xyz="0 0 0.1" rpy="0 0 0"/>
+      <geometry>
+        <cylinder length="0.2" radius="0.01"/>
       </geometry>
       <material name="silver">
@@ -38,6 +44,7 @@
     </visual>
     <collision>
-      <geometry>
-        <cylinder length="0.02" radius="0.01"/>
+      <origin xyz="0 0 0.1" rpy="0 0 0"/>
+      <geometry>
+        <cylinder length="0.2" radius="0.01"/>
       </geometry>
     </collision>
@@ -48,4 +55,20 @@
     </inertial>
   </link>
+  <link name="chassis_link">
+    <visual>
+      <geometry>
+        <box size="${wheelbase_length} ${front_wheelbase_width} ${chassis_height}"/>
+      </geometry>
+    </visual>
+    <collision>
+      <geometry>
+        <box size="${wheelbase_length} ${front_wheelbase_width} ${chassis_height}"/>
+      </geometry>
+    </collision>
+    <inertial>
+      <mass value="${chassis_mass}"/>
+      <box_inertia m="${chassis_mass}" x="${wheelbase_length}" y="${front_wheelbase_width}" z="${chassis_height}"/>
+    </inertial>
+  </link>
   <link name="back_left_wheel">
     <visual>
@@ -91,6 +114,6 @@
     <sensor type="gpu_ray" name="laser_scanner">
       <pose>0 0 0 0 0 0</pose>
-      <visualize>true</visualize>
-      <update_rate>40</update_rate>
+      <visualize>false</visualize>
+      <update_rate>20</update_rate>
       <ray>
         <scan>
@@ -128,5 +151,5 @@
       </geometry>
     </collision>
-    <xacro:cylinder_inertial m="${wheel_mass}" r="${wheel_radius}" h="${wheel_width}"/>
+    <cylinder_inertial m="${wheel_mass}" r="${wheel_radius}" h="${wheel_width}"/>
   </link>
   <link name="front_left_wheel_steer">
@@ -164,5 +187,5 @@
       </geometry>
     </collision>
-    <xacro:cylinder_inertial m="${wheel_mass}" r="${wheel_radius}" h="${wheel_width}"/>
+    <cylinder_inertial m="${wheel_mass}" r="${wheel_radius}" h="${wheel_width}"/>
   </link>
   <link name="front_right_wheel_steer">
@@ -200,5 +223,5 @@
       </geometry>
     </collision>
-    <xacro:cylinder_inertial m="${wheel_mass}" r="${wheel_radius}" h="${wheel_width}"/>
+    <cylinder_inertial m="${wheel_mass}" r="${wheel_radius}" h="${wheel_width}"/>
   </link>
   <joint name="back_left_wheel_joint" type="continuous">
@@ -242,14 +265,23 @@
     <origin rpy="${-pi/2} 0 0" xyz="0 0 0"/>
   </joint>
+  <joint name="chassis_joint" type="fixed">
+    <parent link="base_link"/>
+    <child link="chassis_link"/>
+    <origin rpy="0 0 0" xyz="${wheelbase_length/2} 0 ${chassis_height/2 + chassis_elevation}"/>
+  </joint>
   <gazebo reference="front_left_wheel">
+    <mu1>${wheel_friction}</mu1>
     <material>Gazebo/DarkGrey</material>
   </gazebo>
   <gazebo reference="front_right_wheel">
+    <mu1>${wheel_friction}</mu1>
     <material>Gazebo/DarkGrey</material>
   </gazebo>
   <gazebo reference="back_left_wheel">
+    <mu1>${wheel_friction}</mu1>
     <material>Gazebo/DarkGrey</material>
   </gazebo>
   <gazebo reference="back_right_wheel">
+    <mu1>${wheel_friction}</mu1>
     <material>Gazebo/DarkGrey</material>
   </gazebo>

Commit message: added wheel_diameter parameter

File: fake_car.urdf.xacro (robot description, xacro)
@@ -1,5 +1,6 @@
 <?xml version="1.0"?>
 <robot xmlns:xacro="http://ros.org/wiki/xacro" name="fake_car">
-  <xacro:property name="wheel_radius" value="0.056"/>
+  <xacro:arg name="wheel_diameter" default="0.112"/>
+  <xacro:property name="wheel_radius" value="${$(arg wheel_diameter)/2}"/>
   <xacro:property name="wheel_width" value="0.047"/>
   <xacro:property name="wheel_friction" value="0.8"/>

Commit message: Loose shock

File: fake_car.urdf.xacro (robot description, xacro)
@@ -240,10 +240,39 @@
     <limit effort="10000" velocity="500" />
   </joint>
+  <link name="front_left_wheel_shock">
+      <visual>
+      <origin xyz="0 0 0.1" rpy="0 0 0"/>
+      <geometry>
+        <cylinder length="0.2" radius="0.01"/>
+      </geometry>
+      <material name="silver">
+        <color rgba="0.75 0.75 0.75 1"/>
+      </material>
+    </visual>
+    <collision>
+      <origin xyz="0 0 0.1" rpy="0 0 0"/>
+      <geometry>
+        <cylinder length="0.2" radius="0.01"/>
+      </geometry>
+    </collision>
+    <inertial>
+      <mass value="0.01"/>
+      <inertia ixx="0.015" iyy="0.0375" izz="0.0375"
+               ixy="0" ixz="0" iyz="0"/>
+    </inertial>
+  </link>
+  <joint name="front_left_wheel_shock_joint" type="prismatic">
+    <limit lower="-0.03" upper="0.03"/>
+    <axis xyz="0 0 1"/>
+    <parent link="base_link"/>
+    <child link="front_left_wheel_shock"/>
+    <origin rpy="0 0 0" xyz="${wheelbase_length} ${front_wheelbase_width/2} 0"/>
+  </joint>
   <joint name="front_left_wheel_steer_joint" type="revolute">
     <limit lower="-1" upper="1" effort="1" velocity="5"/>
     <axis xyz="0 0 1"/>
-    <parent link="base_link"/>
+    <parent link="front_left_wheel_shock"/>
     <child link="front_left_wheel_steer"/>
-    <origin rpy="0 0 0" xyz="${wheelbase_length} ${front_wheelbase_width/2} 0"/>
+    <origin rpy="0 0 0" xyz="0 0 0"/>
   </joint>
   <joint name="front_left_wheel_joint" type="continuous">

Commit message: Simple shocks https://youtu.be/NvJLZSEQOmM

File: fake_car.urdf.xacro (robot description, xacro)
@@ -10,4 +10,5 @@
   <xacro:property name="wheel_mass" value="0.1"/>
   <xacro:property name="total_mass" value = "3.0"/>
+  <xacro:property name="shock_travel" value = "0.09"/>
   <xacro:property name="chassis_height" value = "0.06"/>
   <xacro:property name="chassis_elevation" value = "0.03"/>
@@ -226,16 +227,74 @@
     <cylinder_inertial m="${wheel_mass}" r="${wheel_radius}" h="${wheel_width}"/>
   </link>
+  <link name="back_left_wheel_shock">
+      <visual>
+      <origin xyz="0 0 0.1" rpy="0 0 0"/>
+      <geometry>
+        <cylinder length="0.2" radius="0.01"/>
+      </geometry>
+      <material name="silver">
+        <color rgba="0.75 0.75 0.75 1"/>
+      </material>
+    </visual>
+    <collision>
+      <origin xyz="0 0 0.1" rpy="0 0 0"/>
+      <geometry>
+        <cylinder length="0.2" radius="0.01"/>
+      </geometry>
+    </collision>
+    <inertial>
+      <mass value="0.01"/>
+      <inertia ixx="0.015" iyy="0.0375" izz="0.0375"
+               ixy="0" ixz="0" iyz="0"/>
+    </inertial>
+  </link>
+  <joint name="back_left_shock_joint" type="prismatic">
+    <limit lower="${-shock_travel/2}" upper="${shock_travel/2}" effort="100" velocity="100"/>
+    <axis xyz="0 0 1"/>
+    <parent link="base_link"/>
+    <child link="back_left_wheel_shock"/>
+    <origin rpy="0 0 0" xyz="0 ${rear_wheelbase_width/2} 0"/>
+  </joint>
   <joint name="back_left_wheel_joint" type="continuous">
     <axis xyz="0 0 1"/>
-    <parent link="base_link"/>
+    <parent link="back_left_wheel_shock"/>
     <child link="back_left_wheel"/>
-    <origin rpy="${-pi/2} 0 0" xyz="0 ${rear_wheelbase_width/2} 0"/>
+    <origin rpy="${-pi/2} 0 0" xyz="0 0 0"/>
     <limit effort="10000" velocity="500" />
   </joint>
+  <link name="back_right_wheel_shock">
+      <visual>
+      <origin xyz="0 0 0.1" rpy="0 0 0"/>
+      <geometry>
+        <cylinder length="0.2" radius="0.01"/>
+      </geometry>
+      <material name="silver">
+        <color rgba="0.75 0.75 0.75 1"/>
+      </material>
+    </visual>
+    <collision>
+      <origin xyz="0 0 0.1" rpy="0 0 0"/>
+      <geometry>
+        <cylinder length="0.2" radius="0.01"/>
+      </geometry>
+    </collision>
+    <inertial>
+      <mass value="0.01"/>
+      <inertia ixx="0.015" iyy="0.0375" izz="0.0375"
+               ixy="0" ixz="0" iyz="0"/>
+    </inertial>
+  </link>
+  <joint name="back_right_shock_joint" type="prismatic">
+    <limit lower="${-shock_travel/2}" upper="${shock_travel/2}" effort="100" velocity="100"/>
+    <axis xyz="0 0 1"/>
+    <parent link="base_link"/>
+    <child link="back_right_wheel_shock"/>
+    <origin rpy="0 0 0" xyz="0 ${-rear_wheelbase_width/2} 0"/>
+  </joint>
   <joint name="back_right_wheel_joint" type="continuous">
     <axis xyz="0 0 1"/>
-    <parent link="base_link"/>
+    <parent link="back_right_wheel_shock"/>
     <child link="back_right_wheel"/>
-    <origin rpy="${-pi/2} 0 0" xyz="0 ${-rear_wheelbase_width/2} 0.0"/>
+    <origin rpy="${-pi/2} 0 0" xyz="0 0 0"/>
     <limit effort="10000" velocity="500" />
   </joint>
@@ -262,6 +321,35 @@
     </inertial>
   </link>
-  <joint name="front_left_wheel_shock_joint" type="prismatic">
-    <limit lower="-0.03" upper="0.03"/>
+    <link name="front_right_wheel_shock">
+      <visual>
+      <origin xyz="0 0 0.1" rpy="0 0 0"/>
+      <geometry>
+        <cylinder length="0.2" radius="0.01"/>
+      </geometry>
+      <material name="silver">
+        <color rgba="0.75 0.75 0.75 1"/>
+      </material>
+    </visual>
+    <collision>
+      <origin xyz="0 0 0.1" rpy="0 0 0"/>
+      <geometry>
+        <cylinder length="0.2" radius="0.01"/>
+      </geometry>
+    </collision>
+    <inertial>
+      <mass value="0.01"/>
+      <inertia ixx="0.015" iyy="0.0375" izz="0.0375"
+               ixy="0" ixz="0" iyz="0"/>
+    </inertial>
+  </link>
+  <joint name="front_right_shock_joint" type="prismatic">
+    <limit lower="${-shock_travel/2}" upper="${shock_travel/2}" effort="100" velocity="100"/>
+    <axis xyz="0 0 1"/>
+    <parent link="base_link"/>
+    <child link="front_right_wheel_shock"/>
+    <origin rpy="0 0 0" xyz="${wheelbase_length} ${-front_wheelbase_width/2} 0"/>
+  </joint>
+  <joint name="front_left_shock_joint" type="prismatic">
+    <limit lower="${-shock_travel/2}" upper="${shock_travel/2}" effort="100" velocity="100"/>
     <axis xyz="0 0 1"/>
     <parent link="base_link"/>
@@ -285,7 +373,7 @@
     <limit lower="-1" upper="1" effort="1" velocity="5"/>
     <axis xyz="0 0 1"/>
-    <parent link="base_link"/>
+    <parent link="front_right_wheel_shock"/>
     <child link="front_right_wheel_steer"/>
-    <origin rpy="0 0 0" xyz="${wheelbase_length} ${-front_wheelbase_width/2} 0"/>
+    <origin rpy="0 0 0" xyz="0 0 0"/>
   </joint>
   <joint name="front_right_wheel_joint" type="continuous">

Commit message: Added speed curves, adjusted shocks.

File: fake_car.urdf.xacro (robot description, xacro)
@@ -12,5 +12,5 @@
   <xacro:property name="shock_travel" value = "0.09"/>
   <xacro:property name="chassis_height" value = "0.06"/>
-  <xacro:property name="chassis_elevation" value = "0.03"/>
+  <xacro:property name="chassis_elevation" value = "-0.01"/>
   <xacro:property name="chassis_mass" value = "${total_mass-4*wheel_mass}"/>
   <xacro:macro name="cylinder_inertia" params="m r h">
@@ -250,9 +250,9 @@
   </link>
   <joint name="back_left_shock_joint" type="prismatic">
-    <limit lower="${-shock_travel/2}" upper="${shock_travel/2}" effort="100" velocity="100"/>
+    <limit lower="0" upper="${shock_travel}" effort="100" velocity="100"/>
     <axis xyz="0 0 1"/>
     <parent link="base_link"/>
     <child link="back_left_wheel_shock"/>
-    <origin rpy="0 0 0" xyz="0 ${rear_wheelbase_width/2} 0"/>
+    <origin rpy="0 0 0" xyz="0 ${rear_wheelbase_width/2}  ${-shock_travel/2}"/>
   </joint>
   <joint name="back_left_wheel_joint" type="continuous">
@@ -286,9 +286,9 @@
   </link>
   <joint name="back_right_shock_joint" type="prismatic">
-    <limit lower="${-shock_travel/2}" upper="${shock_travel/2}" effort="100" velocity="100"/>
+    <limit lower="0" upper="${shock_travel}" effort="100" velocity="100"/>
     <axis xyz="0 0 1"/>
     <parent link="base_link"/>
     <child link="back_right_wheel_shock"/>
-    <origin rpy="0 0 0" xyz="0 ${-rear_wheelbase_width/2} 0"/>
+    <origin rpy="0 0 0" xyz="0 ${-rear_wheelbase_width/2} ${-shock_travel/2}"/>
   </joint>
   <joint name="back_right_wheel_joint" type="continuous">
@@ -344,16 +344,16 @@
   </link>
   <joint name="front_right_shock_joint" type="prismatic">
-    <limit lower="${-shock_travel/2}" upper="${shock_travel/2}" effort="100" velocity="100"/>
+    <limit lower="0" upper="${shock_travel}" effort="100" velocity="100"/>
     <axis xyz="0 0 1"/>
     <parent link="base_link"/>
     <child link="front_right_wheel_shock"/>
-    <origin rpy="0 0 0" xyz="${wheelbase_length} ${-front_wheelbase_width/2} 0"/>
+    <origin rpy="0 0 0" xyz="${wheelbase_length} ${-front_wheelbase_width/2} ${-shock_travel/2}"/>
   </joint>
   <joint name="front_left_shock_joint" type="prismatic">
-    <limit lower="${-shock_travel/2}" upper="${shock_travel/2}" effort="100" velocity="100"/>
+    <limit lower="0" upper="${shock_travel}" effort="100" velocity="100"/>
     <axis xyz="0 0 1"/>
     <parent link="base_link"/>
     <child link="front_left_wheel_shock"/>
-    <origin rpy="0 0 0" xyz="${wheelbase_length} ${front_wheelbase_width/2} 0"/>
+    <origin rpy="0 0 0" xyz="${wheelbase_length} ${front_wheelbase_width/2}  ${-shock_travel/2}"/>
   </joint>
   <joint name="front_left_wheel_steer_joint" type="revolute">

Commit message: saving, still a little buggy

File: fake_car.urdf.xacro (robot description, xacro)
@@ -35,4 +35,6 @@
     </inertial>
   </xacro:macro>
+  <link name="dummy">
+   </link>
   <link name="base_link">
     <visual>
@@ -249,4 +251,8 @@
     </inertial>
   </link>
+  <joint name="dummy_joint" type="fixed">
+     <parent link="dummy"/>
+     <child link="base_link"/>
+   </joint>
   <joint name="back_left_shock_joint" type="prismatic">
     <limit lower="0" upper="${shock_travel}" effort="100" velocity="100"/>
@@ -388,4 +394,9 @@
     <origin rpy="0 0 0" xyz="${wheelbase_length/2} 0 ${chassis_height/2 + chassis_elevation}"/>
   </joint>
+  <gazebo>
+    <plugin name="gazebo_ros_control" filename="libgazebo_ros_control.so">
+      <robotNamespace>/fake_car</robotNamespace>
+    </plugin>
+  </gazebo>
   <gazebo reference="front_left_wheel">
     <mu1>${wheel_friction}</mu1>
